File: oshe_dmm_KiCAD/oshe_dmm_project_v1/oshe_dmm_project_v1.kicad_pcb (KiCad board)
At the start: 4 copper layers, 101.6 x 177.8 mm, 68 parts, among them J1 FTDI Basic, J2 USB_C_Receptacle_PowerOnly_6P, J3 ON/OFF, J4 Voltage, J5 GND, J6 Current, SW1 PTS526 SK15 SMTR2 LFS, U1 ATmega328P-A, U2 INA219BxD, U3 BQ24075RGT, U5 LM317_SOT-223, U6 ADS1115IDGS, Y1 16MHz

Commit message: Rings ~70% done
updated rings, to be completed tonight
Parts:
- moved R10 3.40 mm to (196.3, 151.5)
- moved R11 3.40 mm to (196.3, 156.9)
- moved R13 3.40 mm to (196.3, 162.4)
Routing:
- net /2V: track 29.8 -> 31.3 mm
Changed lines of the file:
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@@
 		(fp_arc
 			(start 64.20104 22.49932)
-			(mid 64.054479 22.85315)
+			(mid 64.054473 22.853115)
 			(end 63.70066 22.9997)
 			(stroke
@@
 	(footprint "Resistor_SMD:R_1206_3216Metric_Pad1.30x1.75mm_HandSolder"
 		(layer "F.Cu")
-		(at 192.93 162.048 -90)
+		(at 196.315 162.389 -90)
 		(descr "Resistor SMD 1206 (3216 Metric), square (rectangular) end terminal, IPC_7351 nominal with elongated pad for handsoldering. (Body size source: IPC-SM-782 page 72, https://www.pcb-3d.com/wordpress/wp-content/uploads/ipc-sm-782a_amendment_1_and_2.pdf), generated with kicad-footprint-generator")
 		(tags "resistor handsolder")
@@
 	(footprint "Resistor_SMD:R_1206_3216Metric_Pad1.30x1.75mm_HandSolder"
 		(layer "F.Cu")
-		(at 192.93 151.15 -90)
+		(at 196.315 151.491 -90)
 		(descr "Resistor SMD 1206 (3216 Metric), square (rectangular) end terminal, IPC_7351 nominal with elongated pad for handsoldering. (Body size source: IPC-SM-782 page 72, https://www.pcb-3d.com/wordpress/wp-content/uploads/ipc-sm-782a_amendment_1_and_2.pdf), generated with kicad-footprint-generator")
 		(tags "resistor handsolder")
@@
 	(footprint "Resistor_SMD:R_1206_3216Metric_Pad1.30x1.75mm_HandSolder"
 		(layer "F.Cu")
-		(at 192.93 156.587 -90)
+		(at 196.315 156.928 -90)
 		(descr "Resistor SMD 1206 (3216 Metric), square (rectangular) end terminal, IPC_7351 nominal with elongated pad for handsoldering. (Body size source: IPC-SM-782 page 72, https://www.pcb-3d.com/wordpress/wp-content/uploads/ipc-sm-782a_amendment_1_and_2.pdf), generated with kicad-footprint-generator")
 		(tags "resistor handsolder")
@@
 	(gr_circle
 		(center 164.49 152.078)
-		(end 174.49 152.078)
+		(end 189.490112 152.078)
 		(stroke
 			(width 2)
@@
 	(gr_circle
 		(center 164.49 152.078)
-		(end 179.49 152.078)
+		(end 174.49 152.078)
 		(stroke
 			(width 2)
@@
 	(gr_circle
 		(center 164.49 152.078)
-		(end 184.49 152.078)
+		(end 179.49 152.078)
 		(stroke
 			(width 2)
@@
 		(layer "F.Cu")
 	)
+	(gr_arc
+		(start 171.355591 133.293334)
+		(mid 174.515111 134.772014)
+		(end 177.36964 136.777187)
+		(stroke
+			(width 2)
+			(type default)
+		)
+		(layer "F.Cu")
+	)
+	(gr_arc
+		(start 184.19146 148.63527)
+		(mid 184.489977 152.107139)
+		(end 184.181345 155.578124)
+		(stroke
+			(width 2)
+			(type default)
+		)
+		(layer "F.Cu")
+	)
+	(gr_arc
+		(start 179.834186 139.250063)
+		(mid 181.825381 142.103805)
+		(end 183.291804 145.259484)
+		(stroke
+			(width 2)
+			(type default)
+		)
+		(layer "F.Cu")
+	)
 	(gr_line
 		(start 148.488 240.47)
@@
 	)
 	(gr_arc
-		(start 150.389743 146.959687)
-		(mid 151.493044 144.58844)
-		(end 152.991432 142.444865)
+		(start 171.355591 133.293334)
+		(mid 174.515111 134.772014)
+		(end 177.36964 136.777187)
 		(stroke
-			(width 0.1)
+			(width 2)
 			(type default)
 		)
@@
 	)
 	(gr_arc
-		(start 167.092897 137.305071)
-		(mid 167.734534 137.432608)
-		(end 168.37 137.588)
+		(start 164.49 132.078)
+		(mid 166.238117 132.154544)
+		(end 167.972853 132.383591)
 		(stroke
 			(width 0.5)
@@
 	)
 	(gr_arc
-		(start 174.49 152.078)
-		(mid 174.337777 153.816184)
-		(end 173.885744 155.501449)
+		(start 167.972853 132.383591)
+		(mid 169.684178 132.764261)
+		(end 171.355591 133.293334)
 		(stroke
 			(width 0.5)
@@
 	)
 	(gr_arc
-		(start 154.840216 140.593398)
-		(mid 156.983677 139.090717)
-		(end 159.355732 137.983544)
+		(start 168.37 137.588)
+		(mid 164.495001 167.078482)
+		(end 160.600343 137.59059)
 		(stroke
-			(width 0.1)
+			(width 2)
 			(type default)
 		)
@@
 	)
 	(gr_arc
-		(start 173.885744 155.501449)
-		(mid 173.148478 157.081075)
-		(end 172.1481 158.508669)
+		(start 168.837468 127.458911)
+		(mid 170.975549 127.933898)
+		(end 173.063852 128.594196)
+		(stroke
+			(width 0.5)
+			(type default)
+		)
+		(layer "F.Mask")
+	)
+	(gr_arc
+		(start 167.08526 142.420641)
+		(mid 167.505215 142.543409)
+		(end 167.919399 142.684428)
 		(stroke
 			(width 0.1)
@@
 	)
 	(gr_arc
-		(start 174.127591 140.583164)
-		(mid 175.090932 141.465053)
-		(end 175.973912 142.427394)
+		(start 173.063852 128.594197)
+		(mid 186.151091 139.59613)
+		(end 189.107234 156.435951)
 		(stroke
-			(width 0.5)
+			(width 2)
 			(type default)
 		)
@@
 	)
 	(gr_arc
-		(start 152.991431 142.444864)
-		(mid 153.875378 141.478745)
-		(end 154.840216 140.593398)
+		(start 151.642701 136.750023)
+		(mid 154.496384 134.753809)
+		(end 157.653083 133.28288)
 		(stroke
-			(width 0.5)
+			(width 0.1)
 			(type default)
 		)
@@
 	)
 	(gr_arc
-		(start 168.37 137.588)
-		(mid 168.998655 137.77113)
-		(end 169.618719 137.981521)
+		(start 184.19146 148.63527)
+		(mid 184.489977 152.107139)
+		(end 184.181345 155.578124)
 		(stroke
-			(width 0.5)
+			(width 2)
 			(type default)
 		)
@@
 	)
 	(gr_arc
-		(start 178.582584 146.938592)
-		(mid 178.977173 148.187465)
-		(end 179.261319 149.465998)
+		(start 161.030142 132.379539)
+		(mid 162.753513 132.153527)
+		(end 164.49 132.078)
 		(stroke
 			(width 0.5)
@@
 	)
 	(gr_arc
-		(start 161.884844 137.30547)
-		(mid 164.488853 137.077517)
-		(end 167.092897 137.305071)
+		(start 179.834186 139.250063)
+		(mid 181.825381 142.103805)
+		(end 183.291804 145.259484)
 		(stroke
-			(width 0.1)
+			(width 2)
 			(type default)
 		)
@@
 	)
 	(gr_arc
-		(start 179.261318 149.465998)
-		(mid 179.490478 152.070528)
-		(end 179.263913 154.675286)
+		(start 145.693403 145.245149)
+		(mid 147.169742 142.07757)
+		(end 149.174918 139.215333)
 		(stroke
 			(width 0.1)
@@
 	)
 	(gr_arc
-		(start 159.355732 137.983543)
-		(mid 159.973762 137.773525)
-		(end 160.600343 137.590592)
+		(start 157.653083 133.28288)
+		(mid 159.321838 132.757284)
+		(end 161.030142 132.37954)
 		(stroke
 			(width 0.5)
@@
 	)
 	(gr_arc
-		(start 169.618719 137.981522)
-		(mid 171.986874 139.085258)
-		(end 174.127592 140.583163)
+		(start 167.919399 142.684429)
+		(mid 164.486833 162.077995)
+		(end 161.066551 142.682259)
 		(stroke
-			(width 0.1)
+			(width 2)
 			(type default)
 		)
@@
 	)
 	(gr_arc
-		(start 160.600343 137.590591)
-		(mid 161.239466 137.433941)
-		(end 161.884844 137.305471)
+		(start 149.174918 139.215333)
+		(mid 150.35496 137.928774)
+		(end 151.642701 136.750023)
 		(stroke
 			(width 0.5)
@@
 	)
 	(gr_arc
-		(start 175.973912 142.427394)
-		(mid 177.475646 144.568844)
-		(end 178.582584 146.938592)
+		(start 164.49 127.078)
+		(mid 166.672062 127.17341)
+		(end 168.837468 127.458911)
 		(stroke
-			(width 0.1)
+			(width 0.5)
 			(type default)
 		)
@@
 	)
 	(segment
+		(start 209.054 162.803)
+		(end 185.739 162.803)
+		(width 0.2)
+		(layer "B.Cu")
+		(net 60)
+	)
+	(segment
 		(start 180.48 160.588)
 		(end 178.569264 158.677264)
@@
 	)
 	(segment
-		(start 207.543 160.588)
-		(end 180.48 160.588)
+		(start 210.928 160.929)
+		(end 209.054 162.803)
+		(width 0.2)
+		(layer "B.Cu")
+		(net 60)
+	)
+	(segment
+		(start 185.739 162.803)
+		(end 183.865 160.929)
 		(width 0.2)
 		(layer "B.Cu")
